File: mcu.kicad_sch (KiCad schematic)
At the start: 31 parts, among them J4 Conn_01x03_MountingPin, SW1 SW_Push, SW2 SW_Push, U1 RP2350_60QFN, U3 W25Q128JVS, Y1 Crystal_GND24

Commit message: Add testpoints
Parts:
- J4: now left out of the parts list
Changed lines of the file:
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@@
 		(body_style 1)
 		(exclude_from_sim no)
-		(in_bom yes)
+		(in_bom no)
 		(on_board yes)
 		(in_pos_files yes)

Commit message: Fix some bugs in the circuit
Parts:
- added TP4: TestPoint, TestPoint:TestPoint_THTPad_D1.5mm_Drill0.7mm, symbol Connector:TestPoint
Connections:
- net +3.3V: now also TP4.1
- no-connect marks 6 -> 15
Changed lines of the file:
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@@
 	)
 	(junction
+		(at 243.84 24.13)
+		(diameter 0)
+		(color 0 0 0 0)
+	)
+	(junction
 		(at 68.58 25.4)
 		(diameter 0)
@@
 	)
 	(no_connect
+		(at 133.35 101.6)
+	)
+	(no_connect
+		(at 133.35 96.52)
+	)
+	(no_connect
 		(at 133.35 132.08)
 	)
 	(no_connect
+		(at 133.35 114.3)
+	)
+	(no_connect
+		(at 133.35 111.76)
+	)
+	(no_connect
 		(at 133.35 109.22)
 	)
@@
 	)
 	(no_connect
+		(at 133.35 99.06)
+	)
+	(no_connect
 		(at 133.35 124.46)
 	)
+	(no_connect
+		(at 133.35 106.68)
+	)
+	(no_connect
+		(at 133.35 116.84)
+	)
+	(no_connect
+		(at 133.35 104.14)
+	)
+	(no_connect
+		(at 133.35 137.16)
+	)
 	(wire
 		(pts
@@
 	(wire
 		(pts
+			(xy 241.3 24.13) (xy 243.84 24.13)
+		)
+		(stroke
+			(width 0)
+			(type default)
+		)
+	)
+	(wire
+		(pts
 			(xy 161.29 33.02) (xy 161.29 36.83)
 		)
@@
 	(wire
 		(pts
-			(xy 243.84 22.86) (xy 243.84 25.4)
+			(xy 243.84 22.86) (xy 243.84 24.13)
 		)
 		(stroke
@@
 	(wire
 		(pts
+			(xy 243.84 24.13) (xy 243.84 25.4)
+		)
+		(stroke
+			(width 0)
+			(type default)
+		)
+	)
+	(wire
+		(pts
 			(xy 49.53 35.56) (xy 49.53 38.1)
 		)
@@
 					(unit 1)
 				)
+			)
+		)
+	)
+	(symbol
+		(lib_id "Connector:TestPoint")
+		(at 241.3 24.13 90)
+		(unit 1)
+		(body_style 1)
+		(exclude_from_sim no)
+		(in_bom yes)
+		(on_board yes)
+		(in_pos_files yes)
+		(dnp no)
+		(fields_autoplaced yes)
+		(property "Reference" "TP4"
+			(at 237.998 19.05 90)
+			(show_name no)
+			(do_not_autoplace no)
+			(effects
+				(font
+					(size 1.27 1.27)
+				)
+			)
+		)
+		(property "Value" "TestPoint"
+			(at 237.998 21.59 90)
+			(show_name no)
+			(do_not_autoplace no)
+			(effects
+				(font
+					(size 1.27 1.27)
+				)
+			)
+		)
+		(property "Footprint" "TestPoint:TestPoint_THTPad_D1.5mm_Drill0.7mm"
+			(at 241.3 19.05 0)
+			(hide yes)
+			(show_name no)
+			(do_not_autoplace no)
+			(effects
+				(font
+					(size 1.27 1.27)
+				)
+			)
+		)
+		(property "Datasheet" ""
+			(at 241.3 19.05 0)
+			(hide yes)
+			(show_name no)
+			(do_not_autoplace no)
+			(effects
+				(font
+					(size 1.27 1.27)
+				)
+			)
+		)
+		(property "Description" "test point"
+			(at 241.3 24.13 0)
+			(hide yes)
+			(show_name no)
+			(do_not_autoplace no)
+			(effects
+				(font
+					(size 1.27 1.27)
+				)
+			)
+		)
+		(pin "1"
+		)
+		(instances
+			(project "octov1.1"
+				(path "/24892b13-7569-4118-b17c-686e889722f8/aab14ee1-3ec8-4208-96cf-f65e1eb09fc8"
+					(reference "TP4")
+					(unit 1)
+				)
